File: AD_inputs.brd (EAGLE design)
At the start: 250 x 250 mm, 103 parts, among them U1 ANALOG_DEVICES_ADG725BSUZANAL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, X17 6PIN_CON, X18 6PIN_CON

Commit message: Before_autorouting2
Parts:
- moved AN1 162.6 mm to (213.9, 229.1)
- moved RA1 162.6 mm to (213.7, 218.2)
- moved RB1 162.6 mm to (213.7, 210.6)
- moved AN8 160.0 mm to (52.6, 229.1)
- moved RA8 160.0 mm to (52.4, 218.2)
- moved RB8 160.0 mm to (52.4, 210.6)
- moved RA2 116.8 mm to (190.8, 218.2)
- moved RB2 116.8 mm to (190.8, 210.6)
- moved AN2 116.8 mm to (191.0, 229.1)
- moved AN7 114.3 mm to (75.5, 229.1)
- moved RA7 114.3 mm to (75.3, 218.2)
- moved RB7 114.3 mm to (75.3, 210.6)
- moved AN3 68.6 mm to (166.9, 229.1)
- moved AN6 68.6 mm to (98.3, 229.1)
- moved RA3 68.6 mm to (166.7, 218.2)
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Routing:
- net -15V: track 14.8 -> 201.1 mm, vias 0 -> 2
- net A1: track 0.00 -> 184.7 mm
- net A9: track 0.00 -> 155.9 mm, vias 0 -> 4
- net A2: track 0.00 -> 145.2 mm, vias 0 -> 2
- net A10: track 0.00 -> 138.9 mm, vias 0 -> 4
- net A8: track 0.00 -> 124.4 mm, vias 0 -> 2
- net A11: track 0.00 -> 119.5 mm, vias 0 -> 4
- net +3V3: track 539.6 -> 657.6 mm, vias 2 -> 4
- net A3: track 0.00 -> 114.5 mm, vias 0 -> 2
- net A16: track 0.00 -> 111.6 mm, vias 0 -> 2
- net A7: track 0.00 -> 111.0 mm, vias 0 -> 2
- net A6: track 0.00 -> 102.9 mm, vias 0 -> 2
- net A4: track 0.00 -> 99.8 mm, vias 0 -> 2
- net A12: track 0.00 -> 99.7 mm, vias 0 -> 4
- net A5: track 0.00 -> 91.0 mm, vias 0 -> 2
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
Commit message: finished_missing_signature
Routing:
- net SCK: track 0.00 -> 498.6 mm, vias 0 -> 1
- net SS: track 0.00 -> 473.7 mm, vias 0 -> 2
- net MOSI: track 0.00 -> 458.5 mm, vias 0 -> 2
- net DOUT: track 0.00 -> 216.1 mm, vias 0 -> 4
- net AOUT: track 0.00 -> 187.1 mm, vias 0 -> 2
- net D1: track 16.9 -> 195.9 mm, vias 0 -> 2
- net D8: track 18.2 -> 142.7 mm, vias 0 -> 6
- net D2: track 16.9 -> 137.8 mm, vias 0 -> 2
- net D9: track 17.1 -> 135.0 mm, vias 0 -> 2
- net D3: track 18.2 -> 129.4 mm, vias 0 -> 4
- net D7: track 18.2 -> 127.0 mm, vias 0 -> 6
- net D4: track 18.2 -> 125.9 mm, vias 0 -> 4
- net D6: track 18.2 -> 122.2 mm, vias 0 -> 8
- net D10: track 17.0 -> 112.1 mm, vias 0 -> 3
- net D5: track 18.2 -> 106.2 mm, vias 0 -> 4
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
Commit message: final_print
Routing:
- net D2: track 137.8 -> 137.1 mm
Other:
- board text added: "Srylab 03/2022 AD_inputs Jacopo De Santis v1.0"

Commit message: size_error_fixing
Parts:
- moved AN2 67.0 mm to (174.6, 164.2)
- moved AN3 67.0 mm to (150.4, 164.2)
- moved AN4 67.0 mm to (127.6, 164.2)
- moved AN5 67.0 mm to (104.7, 164.2)
- moved AN6 67.0 mm to (81.9, 164.2)
- moved AN7 67.0 mm to (59.0, 164.2)
- moved AN1 66.6 mm to (199.0, 164.2)
- moved AN8 66.0 mm to (39.2, 164.5)
- moved RA1 62.9 mm to (201.0, 156.6)
- moved RA2 62.0 mm to (176.6, 157.9)
- moved RA3 62.0 mm to (152.5, 157.9)
- moved RA4 62.0 mm to (129.7, 157.9)
- moved RA5 62.0 mm to (106.8, 157.9)
- moved RA6 62.0 mm to (83.9, 157.9)
- moved RA7 62.0 mm to (61.1, 157.9)
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Routing:
- net SS: track 473.7 -> 358.5 mm, vias 2 -> 4
- net +15V: track 1287.1 -> 1190.7 mm
- net SCK: track 498.6 -> 410.1 mm, vias 1 -> 2
- net MOSI: track 458.5 -> 383.5 mm
- net -15V: track 201.1 -> 136.2 mm, vias 2 -> 3
- net +3V3: track 657.6 -> 605.3 mm, vias 4 -> 6
- net A3: track 114.5 -> 69.6 mm
- net A2: track 145.2 -> 100.3 mm
- net DOUT: track 216.1 -> 173.7 mm, vias 4 -> 2
- net D1: track 195.9 -> 158.2 mm
- net A1: track 184.7 -> 147.1 mm, vias 0 -> 2
- net A5: track 91.0 -> 62.5 mm
- net A4: track 99.8 -> 72.0 mm
- net +5V: track 280.9 -> 255.6 mm
- net D3: track 129.4 -> 104.4 mm
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Other:
- board size 250 x 250 mm -> 200 x 175 mm

Commit message: size_error_fixed1
Parts:
- moved AN9 44.6 mm to (182.4, 112.2)
- moved AN1 44.6 mm to (171.0, 129.4)
- moved RA9 44.6 mm to (185.1, 124.5)
- moved RB1 44.6 mm to (176.4, 121.7)
- moved RA1 44.6 mm to (173.1, 121.8)
- moved RB9 44.6 mm to (187.8, 124.4)
- moved C1 42.8 mm to (180.0, 16.1)
- moved R1 42.6 mm to (171.1, 16.6)
- moved DIG1 42.1 mm to (171.6, 9.04)
- moved C9 36.4 mm to (187.0, 76.5)
- moved DIG9 36.4 mm to (177.4, 86.7)
- moved R9 36.4 mm to (178.3, 76.5)
- moved AN10 5.09 mm to (184.7, 147.2)
- moved C2 2.54 mm to (195.3, 34.6)
- moved DIG2 2.29 mm to (185.0, 25.8)
Routing:
- net A1: track 147.1 -> 57.9 mm
- net +15V: track 1190.7 -> 1125.6 mm, vias 0 -> 3
- net SCK: track 410.1 -> 349.0 mm, vias 2 -> 4
- net A9: track 153.3 -> 102.0 mm
- net D9: track 134.3 -> 91.2 mm
- net MOSI: track 383.5 -> 342.0 mm, vias 2 -> 4
- net SS: track 358.5 -> 321.1 mm, vias 4 -> 6
- net +3V3: track 605.3 -> 639.5 mm, vias 6 -> 8
- net D1: track 158.2 -> 135.0 mm, vias 2 -> 6
- net D10: track 112.1 -> 114.5 mm
- net N$10: track 11.4 -> 13.2 mm
- net D2: track 120.1 -> 118.6 mm
Other:
- board size 200 x 175 mm -> 175 x 175 mm

Commit message: ready_to_print
Parts:
- moved RB15 3.05 mm to (77.3, 156.4)
- moved X18 2.54 mm to (58.2, 123.3)
- moved RB11 1.78 mm to (170.0, 157.7)
- moved RB12 1.78 mm to (148.4, 157.7)
- moved RB13 1.78 mm to (124.5, 157.7)
- moved RB14 1.78 mm to (101.4, 157.7)
- moved RB5 1.78 mm to (109.1, 156.0)
- moved RA9 1.78 mm to (185.1, 122.8)
- moved RB9 1.78 mm to (187.8, 122.6)
- moved RA11 1.78 mm to (167.3, 157.6)
- moved RA12 1.78 mm to (145.7, 157.6)
- moved RA13 1.78 mm to (121.6, 157.6)
- moved RA14 1.78 mm to (98.7, 157.6)
- moved RA2 1.78 mm to (176.6, 156.1)
- moved RA3 1.78 mm to (152.5, 156.1)
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Routing:
- net SCK: track 349.0 -> 353.5 mm
- net +15V: track 1125.6 -> 1128.7 mm
- net -15V: track 136.2 -> 138.7 mm
- net +5V: track 255.6 -> 258.1 mm
- net +3V3: track 639.5 -> 642.0 mm
- net N$9: track 13.7 -> 11.9 mm
- net N$5: track 6.21 -> 7.99 mm
- net N$4: track 6.03 -> 7.81 mm
- net N$3: track 6.03 -> 7.81 mm
- net N$14: track 11.4 -> 9.59 mm
- net N$13: track 11.4 -> 9.59 mm
- net N$12: track 11.4 -> 9.59 mm
- net N$11: track 11.4 -> 9.59 mm
- net N$1: track 6.03 -> 7.81 mm
- net A4: track 72.0 -> 70.3 mm
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
Commit message: production
Parts:
- added TPA, TPA1, TPA2, TPA9, TPB, TPB1, TPB2, TPB9, TPGND: PTR1TP20R, testpad:TP20R
Connections:
- net A1: now also TPB1.TP
- net A2: now also TPB2.TP
- net A9: now also TPB9.TP
- net AOUT: now also TPB.TP
- net D1: now also TPA1.TP
- net D2: now also TPA2.TP
- net D9: now also TPA9.TP
- net DOUT: now also TPA.TP
- net GND: now also TPGND.TP
Routing:
- net DOUT: track 173.7 -> 192.4 mm
- net A9: track 102.8 -> 109.6 mm
- net D1: track 136.3 -> 142.9 mm, vias 6 -> 7
- net AOUT: track 167.3 -> 172.4 mm
- net D2: track 118.6 -> 122.8 mm
- net D9: track 91.2 -> 94.5 mm
- net A2: track 98.6 -> 101.4 mm
- net A1: track 57.9 -> 59.0 mm
- net D5: track 81.2 -> 82.3 mm
- net D7: track 113.5 -> 112.9 mm
- net +5V: track 258.1 -> 257.5 mm
- net +15V: track 1128.7 -> 1129.3 mm
- net D6: track 108.9 -> 109.4 mm
Other:
- board text added: "Srylab 05/2022 A/D Inputs Jacopo De Santis v1.0"
- board text removed: "Srylab 03/2022 AD_inputs Jacopo De Santis v1.0"
