File: AD_inputs.sch (EAGLE design)
At the start: 100 parts, among them U1 ANALOG_DEVICES_ADG725BSUZANAL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, X17 6PIN_CON, X18 6PIN_CON

Commit message: Before_autorouting
Parts:
- added C17, C18, C19: (no value), 1AKarstenLib:C-EU_SMDC1206H/D
Connections:
- net +5V: now also C17.1, C18.1, C19.1
- net GND: now also C17.2, C18.2, C19.2
Changed lines of the file:
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@@
 <part name="+3V19" library="supply1" deviceset="+3V3" device=""/>
 <part name="GND69" library="supply1" deviceset="GND" device=""/>
+<part name="C17" library="1AKarstenLib" deviceset="C-EU_SMD" device="C1206H/D"/>
+<part name="C18" library="1AKarstenLib" deviceset="C-EU_SMD" device="C1206H/D"/>
+<part name="C19" library="1AKarstenLib" deviceset="C-EU_SMD" device="C1206H/D"/>
+<part name="GND70" library="supply1" deviceset="GND" device=""/>
+<part name="GND71" library="supply1" deviceset="GND" device=""/>
+<part name="GND72" library="supply1" deviceset="GND" device=""/>
 </parts>
 <sheets>
@@
 <instance part="P+22" gate="1" x="86.36" y="109.22"/>
 <instance part="GND37" gate="1" x="132.08" y="-38.1" rot="R90"/>
-<instance part="P+23" gate="1" x="81.28" y="-38.1" rot="R90"/>
-<instance part="P+24" gate="1" x="88.9" y="-40.64" rot="R90"/>
+<instance part="P+23" gate="1" x="68.58" y="-38.1" rot="R90"/>
+<instance part="P+24" gate="1" x="83.82" y="-40.64" rot="R90"/>
 <instance part="C1" gate="G$1" x="294.64" y="30.48" rot="R90"/>
 <instance part="R1" gate="G$1" x="276.86" y="30.48" rot="R180"/>
@@
 <instance part="+3V19" gate="G$1" x="424.18" y="-134.62" rot="R90"/>
 <instance part="GND69" gate="1" x="467.36" y="-134.62" rot="R90"/>
+<instance part="C17" gate="G$1" x="91.44" y="-48.26"/>
+<instance part="C18" gate="G$1" x="76.2" y="-45.72"/>
+<instance part="C19" gate="G$1" x="91.44" y="104.14" rot="R90"/>
+<instance part="GND70" gate="1" x="101.6" y="104.14" rot="R90"/>
+<instance part="GND71" gate="1" x="76.2" y="-58.42"/>
+<instance part="GND72" gate="1" x="91.44" y="-58.42"/>
 </instances>
 <busses>
@@
 <pinref part="C16" gate="G$1" pin="2"/>
 <wire x1="459.74" y1="-134.62" x2="464.82" y2="-134.62" width="0.1524" layer="91"/>
+</segment>
+<segment>
+<pinref part="C19" gate="G$1" pin="2"/>
+<pinref part="GND70" gate="1" pin="GND"/>
+<wire x1="99.06" y1="104.14" x2="96.52" y2="104.14" width="0.1524" layer="91"/>
+</segment>
+<segment>
+<pinref part="C18" gate="G$1" pin="2"/>
+<pinref part="GND71" gate="1" pin="GND"/>
+<wire x1="76.2" y1="-55.88" x2="76.2" y2="-50.8" width="0.1524" layer="91"/>
+</segment>
+<segment>
+<pinref part="C17" gate="G$1" pin="2"/>
+<pinref part="GND72" gate="1" pin="GND"/>
+<wire x1="91.44" y1="-55.88" x2="91.44" y2="-53.34" width="0.1524" layer="91"/>
 </segment>
 </net>
@@
 <pinref part="CON1" gate="G$1" pin="1"/>
 <pinref part="P+22" gate="1" pin="+5V"/>
-<wire x1="86.36" y1="106.68" x2="86.36" y2="101.6" width="0.1524" layer="91"/>
+<wire x1="86.36" y1="106.68" x2="86.36" y2="104.14" width="0.1524" layer="91"/>
+<pinref part="C19" gate="G$1" pin="1"/>
+<wire x1="86.36" y1="104.14" x2="86.36" y2="101.6" width="0.1524" layer="91"/>
+<wire x1="86.36" y1="104.14" x2="88.9" y2="104.14" width="0.1524" layer="91"/>
+<junction x="86.36" y="104.14"/>
 </segment>
 <segment>
 <pinref part="U1" gate="G$0" pin="1_VDD"/>
 <pinref part="P+23" gate="1" pin="+5V"/>
-<wire x1="83.82" y1="-38.1" x2="96.52" y2="-38.1" width="0.1524" layer="91"/>
+<wire x1="71.12" y1="-38.1" x2="76.2" y2="-38.1" width="0.1524" layer="91"/>
+<pinref part="C18" gate="G$1" pin="1"/>
+<wire x1="76.2" y1="-38.1" x2="96.52" y2="-38.1" width="0.1524" layer="91"/>
+<wire x1="76.2" y1="-43.18" x2="76.2" y2="-38.1" width="0.1524" layer="91"/>
+<junction x="76.2" y="-38.1"/>
 </segment>
 <segment>
 <pinref part="U1" gate="G$0" pin="2_VDD"/>
 <pinref part="P+24" gate="1" pin="+5V"/>
+<wire x1="86.36" y1="-40.64" x2="91.44" y2="-40.64" width="0.1524" layer="91"/>
+<pinref part="C17" gate="G$1" pin="1"/>
 <wire x1="91.44" y1="-40.64" x2="96.52" y2="-40.64" width="0.1524" layer="91"/>
-</segment>
-</net>
+<wire x1="91.44" y1="-45.72" x2="91.44" y2="-40.64" width="0.1524" layer="91"/>
+<junction x="91.44" y="-40.64"/>
+</segment>
+</net>

Commit message: production
Parts:
- added TPA, TPA1, TPA2, TPA9, TPB, TPB1, TPB2, TPB9, TPGND: PTR1TP20R, testpad:PTR1TP20R
Connections:
- net A1: now also TPB1.TP
- net A2: now also TPB2.TP
- net A9: now also TPB9.TP
- net AOUT: now also TPB.TP
- net D1: now also TPA1.TP
- net D2: now also TPA2.TP
- net D9: now also TPA9.TP
- net DOUT: now also TPA.TP
- net GND: now also TPGND.TP
Other:
- note added: "Srylab 05/2022 A/D Inputs v1.0 Jacopo De Santis"
- moved on the sheet: C1, C10, C11, C12, C13, C14, C15, C16, C19, C2, C3, C4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
